File: hardware/rev3_timer/display.kicad_sch (KiCad schematic)
At the start: 28 parts, among them U10 SN75468, U11 IN-12A/B, U12 IN-12A/B, U13 IN-12A/B, U14 IN-12A/B, U18 74HC164, U19 SN75468, U2 74HC164, U3 74HC164, U4 74HC164, U5 74HC164, U6 SN75468, U7 SN75468, U8 SN75468, U9 SN75468

Commit message: working on placement
Parts:
- added C17: 0.1uF, Capacitor_THT:C_Disc_D3.0mm_W1.6mm_P2.50mm, symbol Device:C_Small
Connections:
- net GND: now also C17.2
- net VCC: now also C17.1
Changed lines of the file:
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@@
   (junction (at 38.1 119.38) (diameter 0) (color 0 0 0 0)
   )
+  (junction (at 67.31 252.73) (diameter 0) (color 0 0 0 0)
+  )
   (junction (at 186.69 113.03) (diameter 0) (color 0 0 0 0)
   )
@@
   )
   (junction (at 66.04 81.28) (diameter 0) (color 0 0 0 0)
+  )
+  (junction (at 67.31 245.11) (diameter 0) (color 0 0 0 0)
   )
   (junction (at 133.35 90.17) (diameter 0) (color 0 0 0 0)
@@
     (stroke (width 0) (type default) (color 0 0 0 0))
   )
+  (wire (pts (xy 78.74 246.38) (xy 78.74 245.11))
+    (stroke (width 0) (type default) (color 0 0 0 0))
+  )
   (wire (pts (xy 157.48 172.72) (xy 157.48 171.45))
     (stroke (width 0) (type default) (color 0 0 0 0))
@@
     (stroke (width 0) (type default) (color 0 0 0 0))
   )
+  (wire (pts (xy 78.74 251.46) (xy 78.74 252.73))
+    (stroke (width 0) (type default) (color 0 0 0 0))
+  )
   (wire (pts (xy 130.81 60.96) (xy 156.21 60.96))
     (stroke (width 0) (type default) (color 0 0 0 0))
@@
     (stroke (width 0) (type default) (color 0 0 0 0))
   )
+  (wire (pts (xy 67.31 245.11) (xy 78.74 245.11))
+    (stroke (width 0) (type default) (color 0 0 0 0))
+  )
   (wire (pts (xy 66.04 76.2) (xy 110.49 76.2))
     (stroke (width 0) (type default) (color 0 0 0 0))
@@
   )
   (wire (pts (xy 130.81 68.58) (xy 156.21 68.58))
+    (stroke (width 0) (type default) (color 0 0 0 0))
+  )
+  (wire (pts (xy 67.31 252.73) (xy 78.74 252.73))
     (stroke (width 0) (type default) (color 0 0 0 0))
   )
@@
     (pin "1")
   )
+  (symbol (lib_id "Device:C_Small") (at 78.74 248.92 0) (unit 1)
+    (in_bom yes) (on_board yes) (fields_autoplaced)
+    (property "Reference" "C17" (id 0) (at 81.28 247.6562 0)
+      (effects (font (size 1.27 1.27)) (justify left))
+    )
+    (property "Value" "0.1uF" (id 1) (at 81.28 250.1962 0)
+      (effects (font (size 1.27 1.27)) (justify left))
+    )
+    (property "Footprint" "Capacitor_THT:C_Disc_D3.0mm_W1.6mm_P2.50mm" (id 2) (at 78.74 248.92 0)
+      (effects (font (size 1.27 1.27)) hide)
+    )
+    (property "Datasheet" "~" (id 3) (at 78.74 248.92 0)
+      (effects (font (size 1.27 1.27)) hide)
+    )
+    (pin "1")
+    (pin "2")
+  )
   (symbol (lib_id "Device:Lamp_Neon") (at 158.75 231.14 0) (unit 1)
